File: feederboard.sch (EAGLE design)
At the start: 19 parts, among them IC1 TINY13V-10SU, J1 CON_HEADER_PRG_AVR_ICSP_ETCH

Commit message: Pullup for reset
Parts:
- added R3: 100k, LL:R-US_R0805
Connections:
- net N$8 renamed VIN
- removed net VCCF: C6.1, C7.1, FB.1, IC1.VCC
- new net VCC: C6.1, C7.1, FB.1, IC1.VCC, R3.1
- net RST: now also R3.2
Changed lines of the file:
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@@
 <part name="JP1" library="pinhead" deviceset="PINHD-2X2" device="/90"/>
 <part name="GND1" library="SparkFun-Aesthetics" deviceset="GND" device=""/>
+<part name="P+1" library="supply1" deviceset="VCC" device=""/>
+<part name="P+2" library="supply1" deviceset="VCC" device=""/>
+<part name="R3" library="LL" deviceset="R-US_" device="R0805" value="100k"/>
 </parts>
 <sheets>
@@
 <instance part="JP1" gate="A" x="45.72" y="121.92"/>
 <instance part="GND1" gate="1" x="-81.28" y="104.14"/>
+<instance part="P+1" gate="VCC" x="-66.04" y="127"/>
+<instance part="P+2" gate="VCC" x="-71.12" y="71.12"/>
+<instance part="R3" gate="G$1" x="-71.12" y="60.96" rot="R270"/>
 </instances>
 <busses>
@@
 <segment>
 <pinref part="J1" gate="J" pin="RST"/>
-<wire x1="-50.8" y1="53.34" x2="-55.88" y2="53.34" width="0.1524" layer="91"/>
-<label x="-55.88" y="53.34" size="1.778" layer="95" rot="R180" xref="yes"/>
+<wire x1="-50.8" y1="53.34" x2="-71.12" y2="53.34" width="0.1524" layer="91"/>
+<label x="-76.2" y="53.34" size="1.778" layer="95" rot="R180" xref="yes"/>
+<pinref part="R3" gate="G$1" pin="2"/>
+<wire x1="-71.12" y1="53.34" x2="-76.2" y2="53.34" width="0.1524" layer="91"/>
+<wire x1="-71.12" y1="53.34" x2="-71.12" y2="55.88" width="0.1524" layer="91"/>
+<junction x="-71.12" y="53.34"/>
 </segment>
 <segment>
@@
 </segment>
 </net>
-<net name="VCCF" class="0">
-<segment>
-<pinref part="IC1" gate="G$1" pin="VCC"/>
-<pinref part="FB" gate="G$1" pin="1"/>
-<wire x1="-43.18" y1="119.38" x2="-53.34" y2="119.38" width="0.1524" layer="91"/>
-<wire x1="-53.34" y1="119.38" x2="-53.34" y2="121.92" width="0.1524" layer="91"/>
-<pinref part="C7" gate="G$1" pin="1"/>
-<wire x1="-53.34" y1="119.38" x2="-78.74" y2="119.38" width="0.1524" layer="91"/>
-<junction x="-53.34" y="119.38"/>
-<pinref part="C6" gate="G$1" pin="1"/>
-<wire x1="-78.74" y1="119.38" x2="-86.36" y2="119.38" width="0.1524" layer="91"/>
-<junction x="-78.74" y="119.38"/>
-</segment>
-</net>
-<net name="N$8" class="0">
+<net name="VIN" class="0">
 <segment>
 <pinref part="JP1" gate="A" pin="1"/>
@@
 </segment>
 </net>
+<net name="VCC" class="0">
+<segment>
+<pinref part="IC1" gate="G$1" pin="VCC"/>
+<pinref part="FB" gate="G$1" pin="1"/>
+<wire x1="-43.18" y1="119.38" x2="-53.34" y2="119.38" width="0.1524" layer="91"/>
+<wire x1="-53.34" y1="119.38" x2="-53.34" y2="121.92" width="0.1524" layer="91"/>
+<pinref part="C7" gate="G$1" pin="1"/>
+<wire x1="-53.34" y1="119.38" x2="-66.04" y2="119.38" width="0.1524" layer="91"/>
+<junction x="-53.34" y="119.38"/>
+<pinref part="C6" gate="G$1" pin="1"/>
+<wire x1="-66.04" y1="119.38" x2="-78.74" y2="119.38" width="0.1524" layer="91"/>
+<wire x1="-78.74" y1="119.38" x2="-86.36" y2="119.38" width="0.1524" layer="91"/>
+<junction x="-78.74" y="119.38"/>
+<pinref part="P+1" gate="VCC" pin="VCC"/>
+<wire x1="-66.04" y1="119.38" x2="-66.04" y2="124.46" width="0.1524" layer="91"/>
+<junction x="-66.04" y="119.38"/>
+</segment>
+<segment>
+<pinref part="R3" gate="G$1" pin="1"/>
+<pinref part="P+2" gate="VCC" pin="VCC"/>
+<wire x1="-71.12" y1="66.04" x2="-71.12" y2="68.58" width="0.1524" layer="91"/>
+</segment>
+</net>

Commit message: Add PTC fuse on 5V rail
Parts:
- added F1: (no value), adafruit:PTCFUSE-1206
Connections:
- new net VR-OUTSM: C4.1, F1.1, IC2.VR-OUTSM
- net 5V: now also F1.2; no longer C4.1, IC2.VR-OUTSM
Changed lines of the file:
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@@
 <part name="P+2" library="supply1" deviceset="VCC" device=""/>
 <part name="R3" library="LL" deviceset="R-US_" device="R0805" value="100k"/>
+<part name="F1" library="adafruit" deviceset="PTCFUSE" device="-1206"/>
 </parts>
 <sheets>
@@
 <instance part="GND7" gate="1" x="-60.96" y="83.82"/>
 <instance part="R2" gate="G$1" x="35.56" y="27.94" rot="R180"/>
-<instance part="SUPPLY5" gate="G$1" x="96.52" y="129.54"/>
+<instance part="SUPPLY5" gate="G$1" x="106.68" y="132.08"/>
 <instance part="IC2" gate="G$1" x="81.28" y="127"/>
 <instance part="GND8" gate="1" x="81.28" y="111.76"/>
@@
 <instance part="P+2" gate="VCC" x="-71.12" y="71.12"/>
 <instance part="R3" gate="G$1" x="-71.12" y="60.96" rot="R270"/>
+<instance part="F1" gate="G$1" x="101.6" y="124.46"/>
 </instances>
 <busses>
@@
 </segment>
 <segment>
+<pinref part="F1" gate="G$1" pin="2"/>
 <pinref part="SUPPLY5" gate="G$1" pin="5V"/>
-<wire x1="96.52" y1="127" x2="96.52" y2="129.54" width="0.1524" layer="91"/>
-<wire x1="93.98" y1="127" x2="96.52" y2="127" width="0.1524" layer="91"/>
-<pinref part="C4" gate="G$1" pin="1"/>
-<junction x="93.98" y="127"/>
-<pinref part="IC2" gate="G$1" pin="VR-OUTSM"/>
-<wire x1="88.9" y1="127" x2="93.98" y2="127" width="0.1524" layer="91"/>
+<wire x1="106.68" y1="132.08" x2="106.68" y2="127" width="0.1524" layer="91"/>
 </segment>
 </net>
@@
 </segment>
 </net>
+<net name="VR-OUTSM" class="0">
+<segment>
+<wire x1="93.98" y1="127" x2="96.52" y2="127" width="0.1524" layer="91"/>
+<pinref part="C4" gate="G$1" pin="1"/>
+<junction x="93.98" y="127"/>
+<pinref part="IC2" gate="G$1" pin="VR-OUTSM"/>
+<wire x1="88.9" y1="127" x2="93.98" y2="127" width="0.1524" layer="91"/>
+<pinref part="F1" gate="G$1" pin="1"/>
+</segment>
+</net>
